Commit message: add ligh 3d model

File: urdf/drone.urdf (robot description, URDF)
Before this commit: robot DJI_M300_RTK, 4 links, 3 joints
Links:
- link body_FLU: geometry visual mesh filename=package://drone_lidar_front/3D/lidar_front_light3D.stl scale=0.001 0.001 0.001
Joints:
- joint fpv_camera_xsens: origin xyz=-0.16739343 -0.00108291 0.15858862 rpy=-2.105748 -1.569829 -0.537213 -> xyz=0 0 -0.20 rpy=-0.0 0.0 0.0
